Commit message: Fixed non critical errors, now works with gazebo 7, ar_track-alvar tags and world added

File: cvg_sim_gazebo/urdf/quadrotor_base.urdf.xacro (robot description, xacro)
@@ -10,9 +10,4 @@
   <xacro:macro name="quadrotor_base_macro">
     <link name="base_link">
-      <inertial>
-        <mass value="1.477" />
-        <origin xyz="0 0 0" />
-        <inertia ixx="0.01152" ixy="0.0" ixz="0.0" iyy="0.01152" iyz="0.0" izz="0.0218" />
-      </inertial>
       <visual>
         <origin xyz="0 0 0" rpy="0 0 0" />
@@ -28,4 +23,15 @@
       </collision>
     </link>
+    <link name="dummy_link">
+	      <inertial>
+        	<mass value="1.477" />
+        	<origin xyz="0 0 0" />
+        	<inertia ixx="0.01152" ixy="0.0" ixz="0.0" iyy="0.01152" iyz="0.0" izz="0.0218" />
+      	      </inertial>
+    </link>
+    <joint name="dummy_joint" type="fixed">
+ 	 <parent link="base_link"/>
+         <child link="dummy_link"/>
+    </joint>
     <gazebo reference="base_link">
       <turnGravityOff>false</turnGravityOff>

File: cvg_sim_gazebo/urdf/sensors/generic_camera.urdf.xacro (robot description, xacro)
@@ -84,5 +84,4 @@
         </plugin>
       </sensor>
-      <turnGravityOff>true</turnGravityOff>
       <material>Gazebo/Blue</material>
     </gazebo>

File: cvg_sim_gazebo/urdf/sensors/sonar_sensor.urdf.xacro (robot description, xacro)
@@ -55,4 +55,7 @@
         <plugin name="gazebo_ros_${name}_controller" filename="libhector_gazebo_ros_sonar.so">
           <gaussianNoise>0.000</gaussianNoise>
+          <offset>0.0 </offset>
+          <drift>0.0</drift>
+	  <driftFrequency>0.0</driftFrequency>
           <topicName>${ros_topic}</topicName>
           <frameId>${name}_link</frameId>

File: cvg_sim_gazebo_plugins/urdf/quadrotor_sensors.urdf.xacro (robot description, xacro)
@@ -23,4 +23,10 @@
         <rateGaussianNoise>0.00 0.00 0.00</rateGaussianNoise>
         <headingDrift>0.0</headingDrift>
+	<headingDriftFrequency>0.0</headingDriftFrequency>
+	<headingOffset>0.0	</headingOffset>
+	<rateDriftFrequency>0 0 0</rateDriftFrequency>
+	<rateOffset>0 0 0</rateOffset>
+	<accelDriftFrequency>0 0 0</accelDriftFrequency>
+	<accelOffset>0 0 0</accelOffset>
         <headingGaussianNoise>0.00</headingGaussianNoise>
       </plugin>
@@ -33,4 +39,5 @@
         <offset>0</offset>
         <drift>0.1</drift>
+	<driftFrequency>0.0</driftFrequency>
         <gaussianNoise>0.5</gaussianNoise>
       </plugin>
@@ -42,4 +49,5 @@
         <offset>0 0 0</offset>
         <drift>0.0 0.0 0.0</drift>
+	<driftFrequency>0.0 0.0 0.0</driftFrequency>
         <gaussianNoise>1.3e-2 1.3e-2 1.3e-2</gaussianNoise>
       </plugin>
@@ -50,8 +58,12 @@
         <topicName>fix</topicName>
         <velocityTopicName>fix_velocity</velocityTopicName>
+	<offset>0 0 0</offset>
         <drift>5.0 5.0 5.0</drift>
+	<driftFrequency>0.0 0.0 0.0</driftFrequency>
         <gaussianNoise>0.1 0.1 0.1</gaussianNoise>
         <velocityDrift>0 0 0</velocityDrift>
+        <velocityDriftFrequency>0 0 0</velocityDriftFrequency>
         <velocityGaussianNoise>0.1 0.1 0.1</velocityGaussianNoise>
+	<velocityOffset>0 0 0</velocityOffset>
       </plugin>
       <plugin name="quadrotor_groundtruth_sim" filename="libgazebo_ros_p3d.so">
